Commit message: Exploration with namespace, Traversability with modified surface normal

File: ros2_ws/src/scout_v2/scout_ros2/scout_description/urdf/depth_cam.xacro (robot description, xacro)
@@ -1,61 +1,63 @@
 <?xml version="1.0"?>
-<robot xmlns:xacro="http://www.ros.org/wiki/xacro" >
-    <joint name="camera_joint" type="fixed">
-        <parent link="base_link"/>
-        <child link="camera_link"/>
-        <origin xyz="0.4 0 0.18" rpy="0 0 0"/>
-    </joint>
-    <link name="camera_link">
-        <visual>
-            <geometry>
-                <box size="0.010 0.03 0.03"/>
-            </geometry>
-        </visual>
-    </link>
-    <joint name="camera_optical_joint" type="fixed">
-        <parent link="camera_link"/>
-        <child link="camera_link_optical"/>
-        <origin xyz="0 0 0" rpy="${-pi/2} 0 ${-pi/2}"/>
-    </joint>
-    <link name="camera_link_optical"></link>
-    <gazebo reference="camera_link">
-        <sensor name="camera" type="depth">
-            <pose> 0 0 0 0 0 0 </pose>
-            <always_on>true</always_on>
-            <visualize>true</visualize>
-            <update_rate>30</update_rate>
-            <camera>
-                <horizontal_fov>1.089</horizontal_fov>
-                <vertical_fov>1.57</vertical_fov>
-                <image>
-                    <width>640</width>
-                    <height>480</height>
-                    <format>B8G8R8</format>
-                </image>
-                <clip>
-                    <near>0.4</near>
-                    <far>200</far>
-                </clip>
-                <noise>
-                    <type>gaussian</type>
-                    <!-- Noise is sampled independently per pixel on each frame.
-                        That pixel's noise value is added to each of its color
-                        channels, which at that point lie in the range [0,1]. -->
-                    <mean>1.2e-4</mean>
-                    <stddev>0.09</stddev>
-                </noise>
-            </camera>
-            <plugin name="camera_controller" filename="libgazebo_ros_camera.so">
-                <frame_name>camera_link_optical</frame_name>
-                <!-- <min_depth>1.2</min_depth>
-                <max_depth>2.4</max_depth> -->
-                <ros>
-                <!-- <namespace>test_cam</namespace> -->
-                    <remapping>/camera/image_raw:=rgb/image</remapping>
-                    <remapping>/camera/camera_info:=rgb/camera_info</remapping>
-                    <remapping>/camera/depth/image_raw:=depth/image</remapping>
-                </ros>
-            </plugin>
-        </sensor>
-    </gazebo>
+<robot xmlns:xacro="http://www.ros.org/wiki/xacro" name="depth_cam">
+    <xacro:macro name="depth_cam" params="robot_namespace">
+        <link name="${robot_namespace}/camera_link">
+            <visual>
+                <geometry>
+                    <box size="0.010 0.03 0.03"/>
+                </geometry>
+            </visual>
+        </link>
+        <joint name="${robot_namespace}/camera_joint" type="fixed">
+            <parent link="${robot_namespace}/base_link"/>
+            <child link="${robot_namespace}/camera_link"/>
+            <origin xyz="0.4 0 0.18" rpy="0 0 0"/>
+        </joint>
+        <joint name="${robot_namespace}/camera_optical_joint" type="fixed">
+            <parent link="${robot_namespace}/camera_link"/>
+            <child link="${robot_namespace}/camera_link_optical"/>
+            <origin xyz="0 0 0" rpy="${-pi/2} 0 ${-pi/2}"/>
+        </joint>
+        <link name="${robot_namespace}/camera_link_optical"></link>
+        <gazebo reference="${robot_namespace}/camera_link">
+            <sensor name="camera" type="depth">
+                <pose> 0 0 0 0 0 0 </pose>
+                <always_on>true</always_on>
+                <visualize>true</visualize>
+                <update_rate>30</update_rate>
+                <camera>
+                    <horizontal_fov>1.089</horizontal_fov>
+                    <vertical_fov>1.57</vertical_fov>
+                    <image>
+                        <width>640</width>
+                        <height>480</height>
+                        <format>B8G8R8</format>
+                    </image>
+                    <clip>
+                        <near>0.4</near>
+                        <far>200</far>
+                    </clip>
+                    <noise>
+                        <type>gaussian</type>
+                        <!-- Noise is sampled independently per pixel on each frame.
+                            That pixel's noise value is added to each of its color
+                            channels, which at that point lie in the range [0,1]. -->
+                        <mean>1.2e-4</mean>
+                        <stddev>0.09</stddev>
+                    </noise>
+                </camera>
+                <plugin name="camera_controller" filename="libgazebo_ros_camera.so">
+                    <frame_name>${robot_namespace}/camera_link_optical</frame_name>
+                    <!-- <min_depth>1.2</min_depth>
+                    <max_depth>2.4</max_depth> -->
+                    <ros>
+                        <namespace>${robot_namespace}</namespace>
+                        <!-- <remapping>/${robot_namespace}/camera/image_raw:=/${robot_namespace}/rgb/image</remapping>
+                        <remapping>/${robot_namespace}/camera/camera_info:=/${robot_namespace}/rgb/camera_info</remapping>
+                        <remapping>/${robot_namespace}/camera/depth/image_raw:=/${robot_namespace}/depth/image</remapping> -->
+                    </ros>
+                </plugin>
+            </sensor>
+        </gazebo>
+    </xacro:macro>
 </robot>

File: ros2_ws/src/scout_v2/scout_ros2/scout_description/urdf/scout_v2.urdf (robot description, URDF)
Before this commit: robot scout_v2, 13 links, 12 joints
Links:
- removed link base_footprint
- removed link base_link
- removed link camera_link
- removed link camera_link_optical
- removed link front_left_wheel_link
- removed link front_right_wheel_link
- removed link gps_link
- removed link imu_link
- removed link inertial_link
- removed link rear_left_wheel_link
- removed link rear_right_wheel_link
- removed link velodyne
- removed link velodyne_base_link
- added link scout_ns_base_footprint
- added link scout_ns_base_link; collision box size=0.15416666666666667 0.627 0.06999999999999999; collision box size=0.925 0.38 0.21
- added link scout_ns_camera_link; visual box size=0.010 0.03 0.03
- added link scout_ns_camera_link_optical
- added link scout_ns_front_left_wheel_link, mass 3; collision cylinder length=0.11653 radius=0.16459; visual mesh filename=file:///root/ros2_ws/install/scout_description/share/scout_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
- added link scout_ns_front_right_wheel_link, mass 3; collision cylinder length=0.11653 radius=0.16459; visual mesh filename=file:///root/ros2_ws/install/scout_description/share/scout_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
- added link scout_ns_gps_link; collision box size=0.05 0.05 0.05; visual box size=0.05 0.05 0.05
- added link scout_ns_imu_link; collision box size=0.05 0.05 0.05; visual box size=0.05 0.05 0.05
- added link scout_ns_inertial_link, mass 40
- added link scout_ns_rear_left_wheel_link, mass 3; collision cylinder length=0.11653 radius=0.16459; visual mesh filename=file:///root/ros2_ws/install/scout_description/share/scout_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
- added link scout_ns_rear_right_wheel_link, mass 3; collision cylinder length=0.11653 radius=0.16459; visual mesh filename=file:///root/ros2_ws/install/scout_description/share/scout_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
- added link scout_ns_velodyne, mass 0.01; collision sphere radius=0; visual mesh filename=package://velodyne_description/meshes/VLP16_scan.dae
- added link scout_ns_velodyne_base_link, mass 0.83; collision cylinder length=0.0717 radius=0.0516; visual mesh filename=package://velodyne_description/meshes/VLP16_base_1.dae
Joints:
- removed joint base_footprint_joint
- removed joint camera_joint
- removed joint camera_optical_joint
- removed joint front_left_wheel
- removed joint front_right_wheel
- removed joint gps_joint
- removed joint imu_joint
- removed joint inertial_joint
- removed joint rear_left_wheel
- removed joint rear_right_wheel
- removed joint velodyne_base_mount_joint
- removed joint velodyne_base_scan_joint
- added joint scout_ns_base_footprint_joint: type fixed, parent scout_ns_base_footprint, child scout_ns_base_link, origin xyz=0 0 0.23479 rpy=0 0 0
- added joint scout_ns_camera_joint: type fixed, parent scout_ns_base_link, child scout_ns_camera_link, origin xyz=0.4 0 0.18 rpy=0 0 0
- added joint scout_ns_camera_optical_joint: type fixed, parent scout_ns_camera_link, child scout_ns_camera_link_optical, origin xyz=0 0 0 rpy=-1.5707963267948966 0 -1.5707963267948966
- added joint scout_ns_front_left_wheel: type continuous, parent scout_ns_base_link, child scout_ns_front_left_wheel_link, origin xyz=0.249 0.29153 -0.0702 rpy=3.14 0 0, axis 0 -1 0
- added joint scout_ns_front_right_wheel: type continuous, parent scout_ns_base_link, child scout_ns_front_right_wheel_link, origin xyz=0.249 -0.29153 -0.0702 rpy=3.14 0 0, axis 0 -1 0
- added joint scout_ns_gps_joint: type fixed, parent scout_ns_base_link, child scout_ns_gps_link, origin xyz=0.10 0 0.05 rpy=0 0 0
- added joint scout_ns_imu_joint: type fixed, parent scout_ns_base_link, child scout_ns_imu_link, origin xyz=0 0 0.01
- added joint scout_ns_inertial_joint: type fixed, parent scout_ns_base_link, child scout_ns_inertial_link, origin xyz=0 0 0 rpy=0 0 0
- added joint scout_ns_rear_left_wheel: type continuous, parent scout_ns_base_link, child scout_ns_rear_left_wheel_link, origin xyz=-0.249 0.29153 -0.0702 rpy=3.14 0 0, axis 0 -1 0
- added joint scout_ns_rear_right_wheel: type continuous, parent scout_ns_base_link, child scout_ns_rear_right_wheel_link, origin xyz=-0.249 -0.29153 -0.0702 rpy=3.14 0 0, axis 0 -1 0
- added joint scout_ns_velodyne_base_mount_joint: type fixed, parent scout_ns_base_link, child scout_ns_velodyne_base_link, origin xyz=0.5 0 0.4 rpy=0 0.7825 0
- added joint scout_ns_velodyne_base_scan_joint: type fixed, parent scout_ns_velodyne_base_link, child scout_ns_velodyne, origin xyz=0 0 0.0377 rpy=0 0 0

File: ros2_ws/src/scout_v2/scout_ros2/scout_description/urdf/scout_v2.xacro (robot description, xacro)
@@ -3,7 +3,11 @@
     xmlns:xacro="http://ros.org/wiki/xacro"
     xmlns:gazebo="http://gazebosim.org">
-    <xacro:arg name="robot_namespace" default="/" />
+    <xacro:arg name="robot_namespace" default="scout_ns" />
+    <xacro:property name="robot_namespace" value="$(arg robot_namespace)" />
     <xacro:include filename="$(find scout_description)/urdf/scout_wheel_type1.xacro" />
     <xacro:include filename="$(find scout_description)/urdf/scout_wheel_type2.xacro" />
+    <xacro:include filename="$(find scout_description)/urdf/depth_cam.xacro" />
+    <xacro:include filename="$(find scout_description)/urdf/imu_gps.xacro" />
+    <xacro:include filename="$(find velodyne_description)/urdf/VLP-16.urdf.xacro"/>
     <!-- Variables -->
     <xacro:property name="M_PI" value="3.14159"/>
@@ -22,12 +26,12 @@
     <xacro:arg name="organize_cloud" default="false"/>
     <xacro:property name="organize_cloud" value="$(arg organize_cloud)" />
-    <link name="base_footprint"/>
-    <joint name="base_footprint_joint" type="fixed">
-        <parent link="base_footprint" />
-        <child link="base_link" />
+    <link name="${robot_namespace}/base_footprint"/>
+    <joint name="${robot_namespace}/base_footprint_joint" type="fixed">
+        <parent link="${robot_namespace}/base_footprint" />
+        <child link="${robot_namespace}/base_link" />
         <origin xyz="0 0 ${-wheel_vertical_offset + wheel_radius}" rpy="0 0 0" />
     </joint>
     <!-- Base link -->
-    <link name="base_link">
+    <link name="${robot_namespace}/base_link">
         <visual>
             <origin xyz="0 0 0" rpy="0 0 0" />
@@ -49,5 +53,5 @@
         </collision>
     </link>
-    <link name="inertial_link">
+    <link name="${robot_namespace}/inertial_link">
         <inertial>
             <mass value="40" />
@@ -56,22 +60,22 @@
         </inertial>
     </link>
-    <joint name="inertial_joint" type="fixed">
+    <joint name="${robot_namespace}/inertial_joint" type="fixed">
         <origin xyz="0 0 0" rpy="0 0 0" />
-        <parent link="base_link" />
-        <child link="inertial_link" />
+        <parent link="${robot_namespace}/base_link" />
+        <child link="${robot_namespace}/inertial_link" />
     </joint>
     <!-- Scout wheel macros -->
     <!-- wheel labeled from 0 to 3, conter-clockwise, starting from front right wheel -->
     <!-- motor 1 and 2 (left side) are mechanically installed in a reversed direction -->
-    <xacro:scout_wheel_type1 wheel_prefix="front_right">
+    <xacro:scout_wheel_type1 wheel_prefix="front_right" robot_namespace="${robot_namespace}">
         <origin xyz="${wheelbase/2} ${-track/2} ${wheel_vertical_offset}" rpy="3.14 0 0" />
     </xacro:scout_wheel_type1>
-    <xacro:scout_wheel_type1 wheel_prefix="rear_right">
+    <xacro:scout_wheel_type1 wheel_prefix="rear_right" robot_namespace="${robot_namespace}">
         <origin xyz="${-wheelbase/2} ${-track/2} ${wheel_vertical_offset}" rpy="3.14 0 0" />
     </xacro:scout_wheel_type1>
-    <xacro:scout_wheel_type1 wheel_prefix="front_left">
+    <xacro:scout_wheel_type1 wheel_prefix="front_left" robot_namespace="${robot_namespace}">
         <origin xyz="${wheelbase/2} ${track/2} ${wheel_vertical_offset}" rpy="3.14 0 0" />
     </xacro:scout_wheel_type1>
-    <xacro:scout_wheel_type1 wheel_prefix="rear_left">
+    <xacro:scout_wheel_type1 wheel_prefix="rear_left" robot_namespace="${robot_namespace}">
         <origin xyz="${-wheelbase/2} ${track/2} ${wheel_vertical_offset}" rpy="3.14 0 0" />
     </xacro:scout_wheel_type1>
@@ -80,5 +84,5 @@
         <plugin>gazebo_ros2_control/GazeboSystem</plugin>
       </hardware>
-      <joint name="front_left_wheel">
+      <joint name="${robot_namespace}/front_left_wheel">
         <command_interface name="velocity">
           <param name="min">-6</param>
@@ -89,5 +93,5 @@
         <state_interface name="effort"/>
       </joint>
-      <joint name="rear_left_wheel">
+      <joint name="${robot_namespace}/rear_left_wheel">
         <command_interface name="velocity">
           <param name="min">-6</param>
@@ -98,5 +102,5 @@
         <state_interface name="effort"/>
       </joint>
-      <joint name="front_right_wheel">
+      <joint name="${robot_namespace}/front_right_wheel">
         <command_interface name="velocity">
           <param name="min">-6</param>
@@ -107,5 +111,5 @@
         <state_interface name="effort"/>
       </joint>
-      <joint name="rear_right_wheel">
+      <joint name="${robot_namespace}/rear_right_wheel">
         <command_interface name="velocity">
           <param name="min">-6</param>
@@ -119,4 +123,5 @@
     <gazebo>
       <plugin filename="libgazebo_ros2_control.so" name="gazebo_ros2_control">
+        <namespace>${robot_namespace}</namespace>
         <robot_param>robot_description</robot_param>
         <robot_param_node>robot_state_publisher</robot_param_node>
@@ -124,14 +129,8 @@
       </plugin>
     </gazebo>
-   <!-- <xacro:include filename="$(find scout_description)/urdf/scout_v2_add_ouster.gazebo" />  -->
-  <!-- <xacro:include filename="$(find scout_description)/urdf/scout_v2_add_OS0-128.gazebo"/> -->
-  <!-- <OS1-64 parent="base_link" name="os1_sensor" hz="10" samples="220">
-    <origin xyz="0 0 1.2" rpy="0 0 0" />
-  </OS1-64> -->
-  <xacro:include filename="$(find scout_description)/urdf/scout_v2_add_imu_gps.gazebo" />
-  <xacro:include filename="$(find velodyne_description)/urdf/VLP-16.urdf.xacro"/>
-  <xacro:VLP-16 parent="base_link" name="velodyne" topic="/velodyne_points" organize_cloud="${organize_cloud}" hz="10" samples="440" gpu="${gpu}">
-    <origin xyz="0.5 0 0.4" rpy="0 0.7825 0" />
-  </xacro:VLP-16>
-  <xacro:include filename="depth_cam.xacro"/>
+    <xacro:depth_cam robot_namespace="${robot_namespace}"/>
+    <xacro:imu_gps robot_namespace="${robot_namespace}"/>
+    <xacro:VLP-16 parent="${robot_namespace}/base_link" name="${robot_namespace}/velodyne" topic="/${robot_namespace}/velodyne_points" organize_cloud="${organize_cloud}" hz="10" samples="440" gpu="${gpu}">
+      <origin xyz="0.5 0 0.4" rpy="0 0.7825 0" />
+    </xacro:VLP-16>
 </robot>

File: ros2_ws/src/scout_v2/scout_ros2/scout_description/urdf/scout_wheel_type1.xacro (robot description, xacro)
@@ -24,6 +24,6 @@
 -->
 <robot xmlns:xacro="http://ros.org/wiki/xacro" name="scout_wheel">
-    <xacro:macro name="scout_wheel_type1" params="wheel_prefix *joint_pose">
-        <link name="${wheel_prefix}_wheel_link">
+    <xacro:macro name="scout_wheel_type1" params="robot_namespace wheel_prefix *joint_pose">
+        <link name="${robot_namespace}/${wheel_prefix}_wheel_link">
             <inertial>
                 <mass value="3" />
@@ -44,11 +44,11 @@
             </collision>
         </link>
-        <joint name="${wheel_prefix}_wheel" type="continuous">
-            <parent link="base_link"/>
-            <child link="${wheel_prefix}_wheel_link"/>
+        <joint name="${robot_namespace}/${wheel_prefix}_wheel" type="continuous">
+            <parent link="${robot_namespace}/base_link"/>
+            <child link="${robot_namespace}/${wheel_prefix}_wheel_link"/>
             <xacro:insert_block name="joint_pose"/>
             <axis xyz="0 -1 0" rpy="0 0 0" />
         </joint>
-        <gazebo reference="${wheel_prefix}_wheel_link">
+        <gazebo reference="${robot_namespace}/${wheel_prefix}_wheel_link">
             <collision>
                 <surface>

File: ros2_ws/src/scout_v2/scout_ros2/scout_description/urdf/scout_wheel_type2.xacro (robot description, xacro)
@@ -24,6 +24,6 @@
 -->
 <robot xmlns:xacro="http://ros.org/wiki/xacro" name="scout_wheel">
-    <xacro:macro name="scout_wheel_type2" params="wheel_prefix *joint_pose">
-        <link name="${wheel_prefix}_wheel_link">
+    <xacro:macro name="scout_wheel_type2" params="robot_namespace wheel_prefix *joint_pose">
+        <link name="${robot_namespace}/${wheel_prefix}_wheel_link">
             <inertial>
                 <mass value="3" />
@@ -44,11 +44,11 @@
             </collision>
         </link>
-        <joint name="${wheel_prefix}_wheel" type="continuous">
-            <parent link="base_link"/>
-            <child link="${wheel_prefix}_wheel_link"/>
+        <joint name="${robot_namespace}/${wheel_prefix}_wheel" type="continuous">
+            <parent link="${robot_namespace}/base_link"/>
+            <child link="${robot_namespace}/${wheel_prefix}_wheel_link"/>
             <xacro:insert_block name="joint_pose"/>
             <axis xyz="0 -1 0" rpy="0 0 0" />
         </joint>
-        <gazebo reference="${wheel_prefix}_wheel_link">
+        <gazebo reference="${robot_namespace}/${wheel_prefix}_wheel_link">
             <collision>
                 <surface>

Commit message: ORB-SLAM3

File: ros2_ws/src/scout_v2/scout_ros2/scout_description/urdf/depth_cam.xacro (robot description, xacro)
@@ -49,4 +49,14 @@
                 <plugin name="camera_controller" filename="libgazebo_ros_camera.so">
                     <frame_name>${robot_namespace}/camera_link_optical</frame_name>
+                    <hackBaseline>0.07</hackBaseline>
+                    <!-- Projection matrix principal point cx-->
+                    <!-- <P_cx>0</P_cx> -->
+                    <!-- Projection matrix principal point cy-->
+                    <P_cy>380.5</P_cy>
+                    <!-- Projection matrix focal length fy-->
+                    <!-- <P_fy>0</P_fy> -->
+                    <!-- Projection matrix translation Tx, Ty between stereo cameras-->
+                    <Tx>243.5</Tx>
+                    <!-- <Ty>0</Ty> -->
                     <!-- <min_depth>1.2</min_depth>
                     <max_depth>2.4</max_depth> -->

File: ros2_ws/src/scout_v2/scout_ros2/scout_description/urdf/imu_gps.xacro (robot description, xacro)
@@ -26,5 +26,5 @@
       <parent link="${robot_namespace}/base_link"/>
       <child link="${robot_namespace}/imu_link"/>
-      <origin xyz="0 0 0.01"/>
+      <origin xyz="0 0 0.01" rpy="0 0 0"/>
     </joint>
     <gazebo reference="${robot_namespace}/imu_link">

File: ros2_ws/src/scout_v2/scout_ros2/scout_description/urdf/scout_v2.xacro (robot description, xacro)
@@ -132,5 +132,5 @@
     <xacro:imu_gps robot_namespace="${robot_namespace}"/>
     <xacro:VLP-16 parent="${robot_namespace}/base_link" name="${robot_namespace}/velodyne" topic="/${robot_namespace}/velodyne_points" organize_cloud="${organize_cloud}" hz="10" samples="440" gpu="${gpu}">
-      <origin xyz="0.5 0 0.4" rpy="0 0.7825 0" />
+      <origin xyz="0 0 0.4" rpy="0 0 0" />
     </xacro:VLP-16>
     <xacro:scout_decorate />
