Commit message: Tuned scout to MAX - its now a husky

File: ros2_ws/src/scout_v2/scout_ros2/scout_description/urdf/scout_v2.xacro (robot description, xacro)
@@ -5,9 +5,9 @@
     <xacro:arg name="robot_namespace" default="scout_ns" />
     <xacro:property name="robot_namespace" value="$(arg robot_namespace)" />
-    <xacro:include filename="$(find scout_description)/urdf/scout_wheel_type1.xacro" />
-    <xacro:include filename="$(find scout_description)/urdf/scout_wheel_type2.xacro" />
+    <xacro:include filename="$(find scout_description)/urdf/scout_wheel.xacro" />
     <xacro:include filename="$(find scout_description)/urdf/depth_cam.xacro" />
     <xacro:include filename="$(find scout_description)/urdf/imu_gps.xacro" />
     <xacro:include filename="$(find velodyne_description)/urdf/VLP-16.urdf.xacro"/>
+    <xacro:include filename="$(find scout_description)/urdf/decorations.urdf.xacro" />
     <!-- Variables -->
     <xacro:property name="M_PI" value="3.14159"/>
@@ -61,5 +61,5 @@
     </link>
     <joint name="${robot_namespace}/inertial_joint" type="fixed">
-        <origin xyz="0 0 0" rpy="0 0 0" />
+        <origin xyz="0.10 0 ${-wheel_radius/2}" rpy="0 0 0" />
         <parent link="${robot_namespace}/base_link" />
         <child link="${robot_namespace}/inertial_link" />
@@ -68,15 +68,15 @@
     <!-- wheel labeled from 0 to 3, conter-clockwise, starting from front right wheel -->
     <!-- motor 1 and 2 (left side) are mechanically installed in a reversed direction -->
+    <xacro:scout_wheel_type1 wheel_prefix="front_left" robot_namespace="${robot_namespace}">
+        <origin xyz="${wheelbase/2} ${track/2} ${wheel_vertical_offset}" rpy="0 0 0" />
+    </xacro:scout_wheel_type1>
     <xacro:scout_wheel_type1 wheel_prefix="front_right" robot_namespace="${robot_namespace}">
-        <origin xyz="${wheelbase/2} ${-track/2} ${wheel_vertical_offset}" rpy="3.14 0 0" />
+        <origin xyz="${wheelbase/2} ${-track/2} ${wheel_vertical_offset}" rpy="0 0 0" />
+    </xacro:scout_wheel_type1>
+    <xacro:scout_wheel_type1 wheel_prefix="rear_left" robot_namespace="${robot_namespace}">
+        <origin xyz="${-wheelbase/2} ${track/2} ${wheel_vertical_offset}" rpy="0 0 0" />
     </xacro:scout_wheel_type1>
     <xacro:scout_wheel_type1 wheel_prefix="rear_right" robot_namespace="${robot_namespace}">
-        <origin xyz="${-wheelbase/2} ${-track/2} ${wheel_vertical_offset}" rpy="3.14 0 0" />
-    </xacro:scout_wheel_type1>
-    <xacro:scout_wheel_type1 wheel_prefix="front_left" robot_namespace="${robot_namespace}">
-        <origin xyz="${wheelbase/2} ${track/2} ${wheel_vertical_offset}" rpy="3.14 0 0" />
-    </xacro:scout_wheel_type1>
-    <xacro:scout_wheel_type1 wheel_prefix="rear_left" robot_namespace="${robot_namespace}">
-        <origin xyz="${-wheelbase/2} ${track/2} ${wheel_vertical_offset}" rpy="3.14 0 0" />
+        <origin xyz="${-wheelbase/2} ${-track/2} ${wheel_vertical_offset}" rpy="0 0 0" />
     </xacro:scout_wheel_type1>
     <ros2_control name="GazeboSystem" type="system">
@@ -134,3 +134,4 @@
       <origin xyz="0.5 0 0.4" rpy="0 0.7825 0" />
     </xacro:VLP-16>
+    <xacro:scout_decorate />
 </robot>

File: ros2_ws/src/scout_v2/scout_ros2/scout_description/urdf/scout_wheel.xacro (robot description, xacro)
@@ -34,5 +34,5 @@
                 <origin xyz="0 0 0" rpy="0 0 0" />
                 <geometry>
-                    <mesh filename="file://$(find scout_description)/meshes/wheel_type1.dae" />
+                    <mesh filename="file://$(find scout_description)/meshes/wheel.dae" />
                 </geometry>
             </visual>
@@ -44,31 +44,17 @@
             </collision>
         </link>
+        <gazebo reference="${robot_namespace}/${wheel_prefix}_wheel">
+        <mu1 value="1.0"/>
+        <mu2 value="3.5"/>
+        <kp value="10000000.0" />
+        <kd value="1.0" />
+        <fdir1 value="1 0 0"/>
+        </gazebo>
         <joint name="${robot_namespace}/${wheel_prefix}_wheel" type="continuous">
             <parent link="${robot_namespace}/base_link"/>
             <child link="${robot_namespace}/${wheel_prefix}_wheel_link"/>
             <xacro:insert_block name="joint_pose"/>
-            <axis xyz="0 -1 0" rpy="0 0 0" />
+            <axis xyz="0 1 0" rpy="0 0 0" />
         </joint>
-        <gazebo reference="${robot_namespace}/${wheel_prefix}_wheel_link">
-            <collision>
-                <surface>
-                    <friction>
-                        <ode>
-                            <mu>100000.0</mu>
-                            <mu2>100000.0</mu2>
-                            <fdir1>0 0 0</fdir1>
-                            <slip1>0.0</slip1>
-                            <slip2>0.0</slip2>
-                        </ode>
-                    </friction>
-                    <!-- <contact>
-                        <ode>
-                            <kp>1e5</kp>
-                            <kd>1</kd>
-                        </ode>
-                    </contact> -->
-                </surface>
-            </collision>
-        </gazebo>
     </xacro:macro>
 </robot>

Commit message: Verified the working of greedy and random in multirobot

File: ros2_ws/src/scout_v2/scout_ros2/scout_description/urdf/scout_v2.xacro (robot description, xacro)
@@ -132,5 +132,5 @@
     <xacro:imu_gps robot_namespace="${robot_namespace}"/>
     <xacro:VLP-16 parent="${robot_namespace}/base_link" name="${robot_namespace}/velodyne" topic="/${robot_namespace}/velodyne_points" organize_cloud="${organize_cloud}" hz="10" samples="440" gpu="${gpu}">
-      <origin xyz="0 0 0.4" rpy="0 0 0" />
+      <origin xyz="0.5 0 0.4" rpy="0 0.7825 0" />
     </xacro:VLP-16>
     <xacro:scout_decorate />
