Commit message: Fixed the exploration server and BEL

File: ros2_ws/src/velodyne_simulator/velodyne_description/urdf/VLP-16.urdf.xacro (robot description, xacro)
@@ -2,5 +2,5 @@
 <robot xmlns:xacro="http://www.ros.org/wiki/xacro" name="VLP-16">
   <xacro:property name="M_PI" value="3.1415926535897931" />
-  <xacro:macro name="VLP-16" params="*origin parent:=base_link name:=velodyne tf_prefix:='' topic:=/velodyne_points organize_cloud:=false hz:=8 lasers:=16 samples:=1875 collision_range:=0.6 min_range:=0.6 max_range:=5.0 noise:=0.008 min_angle:=-${M_PI} max_angle:=${M_PI} gpu:=false vfov_min:=-0.26 vfov_max:=0.26">
+  <xacro:macro name="VLP-16" params="*origin parent:=base_link name:=velodyne tf_prefix:='' topic:=/velodyne_points organize_cloud:=false hz:=8 lasers:=22 samples:=1875 collision_range:=0.6 min_range:=0.1 max_range:=10.0 noise:=0.008 min_angle:=-${M_PI} max_angle:=${M_PI} gpu:=false vfov_min:=-0.40 vfov_max:=0.40">
     <joint name="${name}_base_mount_joint" type="fixed">
       <xacro:insert_block name="origin" />
